File: circuit/embed/embed.kicad_sch (KiCad schematic)
At the start: 49 parts, among them J1 Downloader, J2 SpekaerSocket, J3 SD_Socket, J4 Display, U1 ESP32-S3-WROOM-2, U2 TPS630701RNMR, U3 LP2950-3.3_TO252, U4 PCM5102A, U5 ATmega328-P, U6 HT82V735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

Commit message: apply
Parts:
- removed R6, R7, R8: R_Variable, symbol Device:R_Variable
- added J5: Conn_01x02_Socket, Connector_PinHeader_2.54mm:PinHeader_1x02_P2.54mm_Vertical, symbol Connector:Conn_01x02_Socket
- added RV1, RV2, RV3: R_Potentiometer_Trim, Potentiometer_SMD:Potentiometer_Bourns_PRS11S_Vertical, symbol Device:R_Potentiometer_Trim
- C10, C12, C17, C19, C20, C4, C5: footprint (none) -> Capacitor_SMD:CP_Elec_4x5.4
- C16, C18: footprint (none) -> Capacitor_SMD:CP_Elec_4x3.9
- R1, R4, R5, R9: footprint (none) -> Resistor_SMD:R_0603_1608Metric
- R2: footprint (none) -> Resistor_SMD:R_2010_5025Metric
- R3: footprint (none) -> Resistor_SMD:R_1210_3225Metric
Connections:
- net Audio: now also RV1.1
- net GND: now also J5.1 (Pin_1), RV1.3, RV2.3, RV3.3
- net R_Audio: now also RV2.1
- net VCC: now also J5.2 (Pin_2)
- net at C19.2: now also RV2.2
- net at C20.2: now also RV1.2
- net at R4.2: now also RV3.1
- net at J2.1 (Pin_1), U6.1 (OUT1): now also RV3.2
Other:
- moved on the sheet: C16, C17, C18, C19, C20, Caux1, Cin1, Cout1, Coutx1, J2, L1, R4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

Commit message: up
Parts:
- removed C14: 0.1u, Capacitor_SMD:C_0402_1005Metric, symbol Device:C
- removed C16, C18: P:0.1u, Capacitor_SMD:CP_Elec_4x3.9, symbol Device:C_Polarized
- C10, C12, C4, C5: footprint Capacitor_SMD:CP_Elec_4x5.4 -> Capacitor_SMD:CP_Elec_3x5.4
Connections:
- net D_LED is gone; now on net +3V3: J4.7 (Pin_7)
- net G0 is gone; now on net BOOT: J1.5 (Pin_5)
- net Audio: now also RV1.3; no longer RV1.1
- net GND: now also RV1.1, RV3.1; no longer RV1.3, RV3.3
- net at R4.2: now also RV3.3; no longer RV3.1
