File: circuit/embed/embed.kicad_pcb (KiCad board)
At the start: 4 copper layers, 86.4 x 53.3 mm, 50 parts, among them J1 Downloader, J2 SpekaerSocket, J3 SD_Socket, J4 Display, J5 Conn_01x02_Socket, U1 ESP32-S3-WROOM-2, U2 TPS630701RNMR, U3 LP2950-3.3_TO252, U4 PCM5102A, U5 ATmega328-P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

Commit message: up
Parts:
- removed C14: 0.1u, Capacitor_SMD:C_0402_1005Metric
- removed C16, C18: P:0.1u, Capacitor_SMD:CP_Elec_4x3.9
- C10, C12, C4, C5: footprint Capacitor_SMD:CP_Elec_4x5.4 -> Capacitor_SMD:CP_Elec_3x5.4
- C8: footprint Capacitor_SMD:C_0504_1310Metric -> Capacitor_SMD:C_0603_1608Metric
- L1: footprint Inductor_SMD:L_Bourns_SRN8040TA -> Inductor_SMD:L_Sunlord_SWPA3015S
- RV1, RV2, RV3: footprint Potentiometer_SMD:Potentiometer_Bourns_PRS11S_Vertical -> Potentiometer_SMD:Potentiometer_Vishay_TS53YJ_Vertical
- Renable1: footprint Resistor_SMD:R_0603_1608Metric -> Resistor_SMD:R_0402_1005Metric
- U1: value ESP32-S3-WROOM-2 -> ESP32-S3-WROOM-1; footprint PCM_Espressif:ESP32-S3-WROOM-2 -> RF_Module:ESP32-S3-WROOM-1
- U3: footprint Package_TO_SOT_SMD:TO-252-2 -> Library:TO-92-3
- U6: footprint 自作:SOP8 -> Package_SO:SSOP-8_3.9x5.05mm_P1.27mm
- moved C13 141.8 mm to (188.0, 51.2), turned to 90 degrees
- moved C15 138.7 mm to (171.8, 26.0)
- moved J2 136.6 mm to (195.7, 73.7), turned to 90 degrees
- moved Y1 136.5 mm to (203.4, 38.2), turned to 180 degrees
- moved RV2 130.6 mm to (183.0, 44.5), turned to 180 degrees
- moved R2 129.4 mm to (190.5, 50.5), turned to 90 degrees
- moved RV3 128.0 mm to (182.0, 70.5), turned to 180 degrees
- moved RV1 127.9 mm to (182.5, 57.2), turned to 180 degrees
- moved C17 122.1 mm to (202.8, 43.5), turned to 180 degrees
- moved C3 112.9 mm to (142.0, 28.0), turned to 90 degrees
- moved C1 110.4 mm to (139.5, 26.8), turned to -90 degrees
- moved R3 110.0 mm to (175.0, 26.0)
- moved U5 108.4 mm to (179.4, 35.0), turned to 90 degrees
- moved C7 106.7 mm to (138.8, 38.2)
- moved C6 106.1 mm to (138.8, 37.2), turned to 180 degrees
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Connections:
- J1 pad 5: G0 -> BOOT
- J4 pad 7: D_LED -> +3V3
- RV1 pad 1: Audio -> GND
- RV1 pad 3: GND -> Audio
- RV3 pad 1: Net-(R4-Pad2) -> GND
- RV3 pad 3: GND -> Net-(R4-Pad2)
Routing:
- net GND: track 0.00 -> 377.3 mm, vias 0 -> 12
- net +5V: track 0.00 -> 185.2 mm, vias 0 -> 4
- net +3V3: track 0.00 -> 105.9 mm, vias 0 -> 6
- net SD_CS: track 0.00 -> 60.8 mm, vias 0 -> 1
- net SD_MOSI: track 0.00 -> 58.5 mm, vias 0 -> 1
- net SD_MISO: track 0.00 -> 56.1 mm, vias 0 -> 1
- net SD_CSK: track 0.00 -> 53.8 mm, vias 0 -> 1
- net Net-(U4-OUTL): track 0.00 -> 53.2 mm, vias 0 -> 2
- net SDA: track 0.00 -> 46.2 mm, vias 0 -> 1
- net D_MOSI: track 0.00 -> 41.4 mm, vias 0 -> 1
- net D_SCK: track 0.00 -> 38.4 mm, vias 0 -> 1
- net SCL: track 0.00 -> 37.8 mm, vias 0 -> 1
- net Net-(U5-PB1): track 0.00 -> 37.1 mm
- net D_RESET: track 0.00 -> 36.9 mm, vias 0 -> 1
- net Net-(J2-Pin_1): track 0.00 -> 36.0 mm
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- added copper zone on F.Cu, net GND

Commit message: up
Parts:
- C10, C12, C4, C5: footprint Capacitor_SMD:CP_Elec_3x5.4 -> Capacitor_SMD:CP_Elec_4x5.4

Commit message: no
Parts:
- U1: value ESP32-S3-WROOM-1 -> ESP32-S3-WROOM-2; footprint RF_Module:ESP32-S3-WROOM-1 -> RF_Module:ESP32-S3-WROOM-2
- moved C9 116.6 mm to (24.8, 42.2)
- moved J2 116.6 mm to (79.7, 61.7)
- moved C1 116.6 mm to (23.5, 14.8)
- moved C10 116.6 mm to (19.8, 46.0)
- moved C11 116.6 mm to (26.8, 41.5)
- moved C12 116.6 mm to (26.5, 46.0)
- moved C13 116.6 mm to (72.0, 39.2)
- moved C15 116.6 mm to (55.8, 14.0)
- moved C17 116.6 mm to (86.8, 31.5)
- moved C19 116.6 mm to (74.5, 28.4)
- moved C2 116.6 mm to (24.8, 14.8)
- moved C20 116.6 mm to (74.5, 44.2)
- moved C3 116.6 mm to (26.0, 16.0)
- moved C4 116.6 mm to (19.5, 29.8)
- moved C5 116.6 mm to (19.5, 22.0)
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Routing:
- net GND: track 377.3 -> 376.5 mm
